File: breadboard-midi.kicad_sch (KiCad schematic)
At the start: 9 parts, among them J1 Conn_02x02_Odd_Even, J2 Conn_02x02_Odd_Even, J4 Conn_01x03, U1 6N137

Commit message: Add image and schematic
Parts:
- D1: value (none) -> 1n4148; footprint (none) -> Diode_THT:D_DO-34_SOD68_P2.54mm_Vertical_KathodeUp
- J3: value (none) -> 3.5mm_Stereo; footprint (none) -> 4ms:EighthInch_PJ398SM
- R1, R2: footprint (none) -> Resistor_THT:R_Axial_DIN0207_L6.3mm_D2.5mm_P2.54mm_Vertical
Changed lines of the file:
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@@
 (kicad_sch (version 20211123) (generator eeschema)
-  (paper "A4")
+  (paper "A5")
   (junction (at 58.42 43.18) (diameter 0) (color 0 0 0 0)
   )
@@
     (in_bom yes) (on_board yes) (fields_autoplaced)
     (property "Reference" "D1" (id 0) (at 123.19 73.66 0))
-    (property "Value" "" (id 1) (at 123.19 76.2 0))
-    (property "Footprint" "" (id 2) (at 123.19 69.85 0)
+    (property "Value" "1n4148" (id 1) (at 123.19 76.2 0))
+    (property "Footprint" "Diode_THT:D_DO-34_SOD68_P2.54mm_Vertical_KathodeUp" (id 2) (at 123.19 69.85 0)
       (effects (font (size 1.27 1.27)) hide)
     )
@@
       (effects (font (size 1.524 1.524)))
     )
-    (property "Value" "" (id 1) (at 98.425 62.23 0)
+    (property "Value" "3.5mm_Stereo" (id 1) (at 98.425 62.23 0)
       (effects (font (size 1.524 1.524)))
     )
-    (property "Footprint" "" (id 2) (at 87.63 91.44 0)
+    (property "Footprint" "4ms:EighthInch_PJ398SM" (id 2) (at 87.63 91.44 0)
       (effects (font (size 1.524 1.524)) (justify left) hide)
     )
@@
       (effects (font (size 1.27 1.27)) (justify right))
     )
-    (property "Footprint" "" (id 2) (at 150.368 60.96 90)
+    (property "Footprint" "Resistor_THT:R_Axial_DIN0207_L6.3mm_D2.5mm_P2.54mm_Vertical" (id 2) (at 150.368 60.96 90)
       (effects (font (size 1.27 1.27)) hide)
     )
@@
     (property "Reference" "R2" (id 0) (at 114.3 58.42 90))
     (property "Value" "220" (id 1) (at 114.3 60.96 90))
-    (property "Footprint" "" (id 2) (at 114.3 66.548 90)
-      (effects (font (size 1.27 1.27)) hide)
-    )
+    (property "Footprint" "Resistor_THT:R_Axial_DIN0207_L6.3mm_D2.5mm_P2.54mm_Vertical" (id 2) (at 114.3 66.548 90)
+      (effects (font (size 1.27 1.27)) hide)
+    )
